Commit message: Add ground to obstacles

File: obstacles.urdf (robot description, URDF)
Before this commit: robot obstacles, 2 links, 0 joints
Links:
- added link ground; collision box size=1.5 1.5 0.1; visual box size=1.5 1.5 0.1

Commit message: Update urdf (copy from gear)

File: obstacles.urdf (robot description, URDF)
Before this commit: robot obstacles, 3 links, 0 joints
Links:
- removed link ground
